File: tpa3130d2_demoboard/tpa3130d2_demoboard.kicad_sch (KiCad schematic)
At the start: 5 parts, among them J1 AudioJack3_Ground_SwitchTR, J2 Conn_01x03_Pin, J3 Screw_Terminal_01x02, J4 Barrel_Jack_MountingPin, U1 TPA3130D2DAPR

Commit message: Split scheme
Parts:
- removed J1: AudioJack3_Ground_SwitchTR, tpa3130d2_demoboard:AudioJack_3.5mm_PJ311, symbol Connector_Audio:AudioJack3_Ground_SwitchTR
- removed J2: Conn_01x03_Pin, Connector_PinHeader_2.54mm:PinHeader_1x03_P2.54mm_Vertical, symbol Connector:Conn_01x03_Pin
- removed J3: Screw_Terminal_01x02, TerminalBlock:TerminalBlock_bornier-2_P5.08mm, symbol Connector:Screw_Terminal_01x02
- removed J4: Barrel_Jack_MountingPin, Connector_BarrelJack:BarrelJack_GCT_DCJ200-10-A_Horizontal, symbol Connector:Barrel_Jack_MountingPin
- removed U1: TPA3130D2DAPR, tpa3130d2_demoboard:TPA3130D2DAPR_M, symbol tpa3130d2_demoboard:TPA3130D2DAPR
Connections:
- no-connect marks 2 -> 0
Other:
- added sheet audio_input (audio_input.kicad_sch)
- added sheet audio_output (audio_output.kicad_sch)
- added sheet tpa3130d2 (tpa3130d2.kicad_sch)

Commit message: Initial PCB layout
Parts:
- added H1, H2, H3, H4: MountingHole, MountingHole:MountingHole_3.2mm_M3, symbol Mechanical:MountingHole
Other:
- note added: "Mounting Holes (M3)"
