File: tpa3130d2_demoboard/audio_output.kicad_sch (KiCad schematic)
At the start: 2 parts, among them J2 Conn_01x03_Pin, J6 Screw_Terminal_01x02

Commit message: Scheme complete
Parts:
- removed J2: Conn_01x03_Pin, Connector_PinHeader_2.54mm:PinHeader_1x03_P2.54mm_Vertical, symbol Connector:Conn_01x03_Pin
- added C300, C301, C308, C309: 220nF, symbol Device:C
- added C302, C303, C310, C311: 1uF, symbol Device:C_Polarized
- added C304, C305, C312, C313: 1nF, symbol Device:C
- added C306, C307, C314, C315: 10nF, symbol Device:C
- added J301: Screw_Terminal_01x02, TerminalBlock:TerminalBlock_bornier-2_P5.08mm, symbol Connector:Screw_Terminal_01x02
- added L300, L301, L302, L303: 10uH, symbol Device:L
- added R300, R301, R303, R304: 3R3, symbol Device:R
- added R302, R305: 47kR, symbol Device:R
- renumbered J6 to J300
Connections:
- net BSNL: now also C309.1
- net BSNR: now also C301.1
- net BSPL: now also C308.1
- net BSPR: now also C300.1
- net GND: now also C302.2, C303.2, C304.2, C305.1, C306.2, C307.2, C310.2, C311.2, C312.2, C313.1, C314.2, C315.2
- net OUTNL: now also C309.2, L303.1
- net OUTNR: now also C301.2, L301.1
- net OUTPL: now also C308.2, L302.1
- net OUTPR: now also C300.2, L300.1
- net OUT_R_P: now reaches J300.1 (Pin_1)
- net OUT_R_P: now also C302.1, C304.1, L300.2, R300.1, R302.1
- net OUT_R_N: now reaches J300.2 (Pin_2)
- net OUT_R_N: now also C303.1, C305.2, L301.2, R301.1, R302.2
- new net: C314.1, R303.2
- new net: C306.1, R300.2
- new net: C307.1, R301.2
- new net: C315.1, R304.2
- new net OUT_L_N: C311.1, C313.2, J301.2 (Pin_2), L303.2, R304.1, R305.2
- new net OUT_L_P: C310.1, C312.1, J301.1 (Pin_1), L302.2, R303.1, R305.1
Other:
- note added: "Optional C-RC EMI Snubber"
- moved on the sheet: J300

Commit message: Fill BOM
Parts:
- C300, C301, C308, C309: footprint (none) -> Capacitor_SMD:C_0603_1608Metric; Manufacturer (none) -> Samsung Electro-Mechanics; Part Number (none) -> CL10B224KA8NNNC
- C302, C303, C310, C311: footprint (none) -> Capacitor_Tantalum_SMD:CP_EIA-3216-18_Kemet-A; Manufacturer (none) -> Kyocera AVX; Part Number (none) -> TAJA105K035RNJ
- C304, C305, C312, C313: footprint (none) -> Capacitor_SMD:C_0603_1608Metric; Manufacturer (none) -> Samsung Electro-Mechanics; Part Number (none) -> CL10B102KB8NNNC
- C306, C307, C314, C315: footprint (none) -> Capacitor_SMD:C_0603_1608Metric; Manufacturer (none) -> Samsung Electro-Mechanics; Part Number (none) -> CL10B104KB8NNNC
- J300, J301: Manufacturer (none) -> Ningbo Kangnex Elec; Part Number (none) -> WJ500V-5.08-2P
- L300, L301, L302, L303: footprint (none) -> Inductor_SMD:L_Wuerth_HCM-7050; Manufacturer (none) -> SHOU HAN; Part Number (none) -> CYA0630-10UH
- R300, R301, R303, R304: Manufacturer (none) -> UNI-ROYAL(Uniroyal Elec); Part Number (none) -> 0603WAF300KT5E
- R302, R305: footprint (none) -> Resistor_SMD:R_0603_1608Metric; Manufacturer (none) -> UNI-ROYAL(Uniroyal Elec); Part Number (none) -> 0603WAJ0473T5E

Commit message: Footprint updates
Parts:
- L300, L301, L302, L303: footprint Inductor_SMD:L_Wuerth_HCM-7050 -> tpa3130d2_demoboard:Inductor_CYA0630-10UH
- R300, R301, R303, R304: footprint (none) -> Resistor_SMD:R_0603_1608Metric
Changed lines of the file:
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@@
 			)
 		)
-		(property "Footprint" "Inductor_SMD:L_Wuerth_HCM-7050"
+		(property "Footprint" "tpa3130d2_demoboard:Inductor_CYA0630-10UH"
 			(at 60.96 33.02 0)
 			(effects
@@
 			)
 		)
-		(property "Footprint" "Inductor_SMD:L_Wuerth_HCM-7050"
+		(property "Footprint" "tpa3130d2_demoboard:Inductor_CYA0630-10UH"
 			(at 60.96 95.25 0)
 			(effects
@@
 			)
 		)
-		(property "Footprint" ""
+		(property "Footprint" "Resistor_SMD:R_0603_1608Metric"
 			(at 97.282 100.33 90)
 			(effects
@@
 			)
 		)
-		(property "Footprint" ""
+		(property "Footprint" "Resistor_SMD:R_0603_1608Metric"
 			(at 97.282 38.1 90)
 			(effects
@@
 			)
 		)
-		(property "Footprint" "Inductor_SMD:L_Wuerth_HCM-7050"
+		(property "Footprint" "tpa3130d2_demoboard:Inductor_CYA0630-10UH"
 			(at 60.96 76.2 0)
 			(effects
@@
 			)
 		)
-		(property "Footprint" ""
+		(property "Footprint" "Resistor_SMD:R_0603_1608Metric"
 			(at 100.838 132.08 90)
 			(effects
@@
 			)
 		)
-		(property "Footprint" "Inductor_SMD:L_Wuerth_HCM-7050"
+		(property "Footprint" "tpa3130d2_demoboard:Inductor_CYA0630-10UH"
 			(at 60.96 138.43 0)
 			(effects
@@
 			)
 		)
-		(property "Footprint" ""
+		(property "Footprint" "Resistor_SMD:R_0603_1608Metric"
 			(at 100.838 69.85 90)
 			(effects

Commit message: Initial PCB layout
Connections:
- net OUT_L_N: now also J301.1 (Pin_1); no longer J301.2 (Pin_2)
- net OUT_L_P: now also J301.2 (Pin_2); no longer J301.1 (Pin_1)
Other:
- moved on the sheet: C308, C309, C310, C311, C312, C313, C314, C315, J301, L302, L303, R303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

Commit message: Minor changes in terminal block footprint
Parts:
- J300, J301: footprint TerminalBlock:TerminalBlock_bornier-2_P5.08mm -> tpa3130d2_demoboard:terminal_block
Connections:
- net OUT_L_N: now also J301.2 (Pin_2); no longer J301.1 (Pin_1)
- net OUT_L_P: now also J301.1 (Pin_1); no longer J301.2 (Pin_2)
- net OUT_R_N: now also J300.1 (Pin_1); no longer J300.2 (Pin_2)
- net OUT_R_P: now also J300.2 (Pin_2); no longer J300.1 (Pin_1)
Changed lines of the file:
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@@
 	(wire
 		(pts
-			(xy 69.85 95.25) (xy 85.09 95.25)
+			(xy 134.62 54.61) (xy 139.7 54.61)
 		)
 		(stroke
@@
 	(wire
 		(pts
-			(xy 53.34 138.43) (xy 57.15 138.43)
+			(xy 69.85 95.25) (xy 85.09 95.25)
 		)
 		(stroke
@@
 	(wire
 		(pts
-			(xy 63.5 54.61) (xy 69.85 54.61)
+			(xy 53.34 138.43) (xy 57.15 138.43)
 		)
 		(stroke
@@
 	(wire
 		(pts
-			(xy 85.09 76.2) (xy 99.06 76.2)
+			(xy 63.5 54.61) (xy 69.85 54.61)
 		)
 		(stroke
@@
 	(wire
 		(pts
-			(xy 85.09 138.43) (xy 85.09 134.62)
+			(xy 85.09 76.2) (xy 99.06 76.2)
 		)
 		(stroke
@@
 	(wire
 		(pts
-			(xy 114.3 76.2) (xy 134.62 76.2)
+			(xy 85.09 138.43) (xy 85.09 134.62)
 		)
 		(stroke
@@
 	(wire
 		(pts
-			(xy 99.06 138.43) (xy 99.06 137.16)
+			(xy 114.3 76.2) (xy 134.62 76.2)
 		)
 		(stroke
@@
 	(wire
 		(pts
-			(xy 134.62 116.84) (xy 139.7 116.84)
+			(xy 99.06 138.43) (xy 99.06 137.16)
 		)
 		(stroke
@@
 	(wire
 		(pts
-			(xy 134.62 54.61) (xy 139.7 54.61)
+			(xy 85.09 138.43) (xy 99.06 138.43)
 		)
 		(stroke
@@
 	(wire
 		(pts
-			(xy 85.09 138.43) (xy 99.06 138.43)
+			(xy 99.06 106.68) (xy 99.06 105.41)
 		)
 		(stroke
@@
 	(wire
 		(pts
-			(xy 99.06 106.68) (xy 99.06 105.41)
+			(xy 63.5 116.84) (xy 69.85 116.84)
 		)
 		(stroke
@@
 	(wire
 		(pts
-			(xy 63.5 116.84) (xy 69.85 116.84)
+			(xy 99.06 95.25) (xy 99.06 97.79)
 		)
 		(stroke
@@
 	(wire
 		(pts
-			(xy 99.06 95.25) (xy 99.06 97.79)
+			(xy 134.62 114.3) (xy 139.7 114.3)
 		)
 		(stroke
@@
 	(wire
 		(pts
-			(xy 99.06 116.84) (xy 99.06 114.3)
+			(xy 134.62 116.84) (xy 139.7 116.84)
 		)
 		(stroke
@@
 	(wire
 		(pts
-			(xy 85.09 127) (xy 85.09 116.84)
+			(xy 99.06 116.84) (xy 99.06 114.3)
 		)
 		(stroke
@@
 	(wire
 		(pts
-			(xy 85.09 54.61) (xy 85.09 66.04)
+			(xy 85.09 127) (xy 85.09 116.84)
 		)
 		(stroke
@@
 	(wire
 		(pts
-			(xy 69.85 116.84) (xy 69.85 105.41)
+			(xy 85.09 54.61) (xy 85.09 66.04)
 		)
 		(stroke
@@
 	(wire
 		(pts
-			(xy 34.29 138.43) (xy 40.64 138.43)
+			(xy 69.85 116.84) (xy 69.85 105.41)
 		)
 		(stroke
@@
 	(wire
 		(pts
-			(xy 85.09 95.25) (xy 85.09 97.79)
+			(xy 34.29 138.43) (xy 40.64 138.43)
 		)
 		(stroke
@@
 	(wire
 		(pts
-			(xy 69.85 138.43) (xy 85.09 138.43)
+			(xy 85.09 95.25) (xy 85.09 97.79)
 		)
 		(stroke
@@
 	(wire
 		(pts
-			(xy 134.62 114.3) (xy 139.7 114.3)
+			(xy 69.85 138.43) (xy 85.09 138.43)
 		)
 		(stroke
@@
 	(wire
 		(pts
-			(xy 134.62 57.15) (xy 139.7 57.15)
+			(xy 114.3 33.02) (xy 114.3 50.8)
 		)
 		(stroke
@@
 	(wire
 		(pts
-			(xy 114.3 33.02) (xy 114.3 50.8)
+			(xy 34.29 33.02) (xy 40.64 33.02)
 		)
 		(stroke
@@
 	(wire
 		(pts
-			(xy 34.29 33.02) (xy 40.64 33.02)
+			(xy 64.77 95.25) (xy 69.85 95.25)
 		)
 		(stroke
@@
 	(wire
 		(pts
-			(xy 64.77 95.25) (xy 69.85 95.25)
+			(xy 134.62 57.15) (xy 139.7 57.15)
 		)
 		(stroke
@@
 	(symbol
 		(lib_id "Connector:Screw_Terminal_01x02")
-		(at 144.78 114.3 0)
+		(at 144.78 116.84 0)
+		(mirror x)
 		(unit 1)
 		(exclude_from_sim no)
@@
 		(dnp no)
 		(property "Reference" "J301"
-			(at 144.78 123.19 0)
+			(at 144.78 107.95 0)
 			(effects
 				(font
@@
 		)
 		(property "Value" "Screw_Terminal_01x02"
-			(at 144.78 120.65 0)
+			(at 144.78 110.49 0)
 			(effects
 				(font
@@
 			)
 		)
-		(property "Footprint" "TerminalBlock:TerminalBlock_bornier-2_P5.08mm"
-			(at 144.78 114.3 0)
+		(property "Footprint" "tpa3130d2_demoboard:terminal_block"
+			(at 144.78 116.84 0)
 			(effects
 				(font
@@
 		)
 		(property "Datasheet" "~"
-			(at 144.78 114.3 0)
+			(at 144.78 116.84 0)
 			(effects
 				(font
@@
 		)
 		(property "Description" "Generic screw terminal, single row, 01x02, script generated (kicad-library-utils/schlib/autogen/connector/)"
-			(at 144.78 114.3 0)
+			(at 144.78 116.84 0)
 			(effects
 				(font
@@
 		)
 		(property "Manufacturer" "Ningbo Kangnex Elec"
-			(at 144.78 114.3 0)
+			(at 144.78 116.84 0)
 			(effects
 				(font
@@
 		)
 		(property "Part Number" "WJ500V-5.08-2P"
-			(at 144.78 114.3 0)
+			(at 144.78 116.84 0)
 			(effects
 				(font
@@
 	(symbol
 		(lib_id "Connector:Screw_Terminal_01x02")
-		(at 144.78 54.61 0)
+		(at 144.78 57.15 0)
+		(mirror x)
 		(unit 1)
 		(exclude_from_sim no)
@@
 		(dnp no)
 		(property "Reference" "J300"
-			(at 144.78 63.5 0)
+			(at 144.78 48.26 0)
 			(effects
 				(font
@@
 		)
 		(property "Value" "Screw_Terminal_01x02"
-			(at 144.78 60.96 0)
+			(at 144.78 50.8 0)
 			(effects
 				(font
@@
 			)
 		)
-		(property "Footprint" "TerminalBlock:TerminalBlock_bornier-2_P5.08mm"
-			(at 144.78 54.61 0)
+		(property "Footprint" "tpa3130d2_demoboard:terminal_block"
+			(at 144.78 57.15 0)
 			(effects
 				(font
@@
 		)
 		(property "Datasheet" "~"
-			(at 144.78 54.61 0)
+			(at 144.78 57.15 0)
 			(effects
 				(font
@@
 		)
 		(property "Description" "Generic screw terminal, single row, 01x02, script generated (kicad-library-utils/schlib/autogen/connector/)"
-			(at 144.78 54.61 0)
+			(at 144.78 57.15 0)
 			(effects
 				(font
@@
 		)
 		(property "Manufacturer" "Ningbo Kangnex Elec"
-			(at 144.78 54.61 0)
+			(at 144.78 57.15 0)
 			(effects
 				(font
@@
 		)
 		(property "Part Number" "WJ500V-5.08-2P"
-			(at 144.78 54.61 0)
+			(at 144.78 57.15 0)
 			(effects
 				(font
